Commit message: change Ubuntu20

File: cube_petit_description/urdf/sensors/lidar.xacro (robot description, xacro)
@@ -4,5 +4,5 @@
     <parent link="body_link"/>
     <child link="pacecat_link"/>
-    <origin rpy="0 0 3.14159" xyz="0.0 0 0.23975"/>
+    <origin rpy="0 0 0" xyz="0.0 0 0.23975"/>
   </joint>
   <link name="pacecat_link">
